Commit message: mpc_wbic done

File: example/cpp/robots/h1_description/urdf/h1.urdf (robot description, URDF)
Before this commit: robot h1_description, 26 links, 25 joints
Links:
- added link left_front_dummy_link, mass 0
- added link left_rear_dummy_link
- added link right_front_dummy_link
- added link right_rear_dummy_link
Joints:
- added joint left_front_joint: type fixed, parent left_ankle_link, child left_front_dummy_link, origin xyz=0.2 0 -0.06 rpy=0 0 0, axis 0 1 0
- added joint left_rear_joint: type fixed, parent left_ankle_link, child left_rear_dummy_link, origin xyz=-0.1 0 -0.06 rpy=0 0 0, axis 0 1 0
- added joint right_front_joint: type fixed, parent right_ankle_link, child right_front_dummy_link, origin xyz=0.2 0 -0.06 rpy=0 0 0, axis 0 1 0
- added joint right_rear_joint: type fixed, parent right_ankle_link, child right_rear_dummy_link, origin xyz=-0.1 0 -0.06 rpy=0 0 0, axis 0 1 0
